File: snowbackpack.kicad_sch (KiCad schematic)
At the start: 86 parts, among them J10 Conn_01x01_Pin, J11 Conn_01x01_Pin, J13 Conn_01x01_Pin, J2 Conn_01x01_Pin, J3 Conn_01x01_Pin, J4 Conn_01x01_Pin, J5 Conn_01x01_Pin, J6 Conn_01x01_Pin, J7 Conn_01x01_Pin, J8 Conn_01x01_Pin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

Commit message: Updated BOM
Parts:
- D2: value PTVS5V0Z1USK -> KLXES15AAA1
- D4: value D_Schottky -> RB161QS-40T18R
- TP5, TP6, TP8, TP9: now left out of the parts list
Other:
- note removed: "check footprint and model"
Changed lines of the file:
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@@
 		)
 	)
-	(text "check footprint and model"
-		(exclude_from_sim no)
-		(at 248.158 216.916 0)
-		(effects
-			(font
-				(size 1.27 1.27)
-			)
-		)
-	)
 	(junction
 		(at 76.2 114.3)
@@
 		(unit 1)
 		(exclude_from_sim no)
-		(in_bom yes)
+		(in_bom no)
 		(on_board yes)
 		(dnp no)
@@
 		(unit 1)
 		(exclude_from_sim no)
-		(in_bom yes)
+		(in_bom no)
 		(on_board yes)
 		(dnp no)
@@
 			)
 		)
-		(property "Value" "PTVS5V0Z1USK"
+		(property "Value" "KLXES15AAA1"
 			(at 256.54 209.042 0)
 			(effects
@@
 		(unit 1)
 		(exclude_from_sim no)
-		(in_bom yes)
+		(in_bom no)
 		(on_board yes)
 		(dnp no)
@@
 			)
 		)
-		(property "Value" "D_Schottky"
+		(property "Value" "RB161QS-40T18R"
 			(at 49.53 209.2324 90)
 			(effects
@@
 		(unit 1)
 		(exclude_from_sim no)
-		(in_bom yes)
+		(in_bom no)
 		(on_board yes)
 		(dnp no)
